Commit message: cleaned up the lidar implementation. added a logo.

File: hermes_create_description/urdf/create3.urdf.xacro (robot description, xacro)
@@ -26,4 +26,6 @@
   <xacro:property name="caster_position_x"       value="${12.5*cm2m}" />
   <xacro:property name="caster_position_z"       value="${-5.55*cm2m}" />
+  <xacro:property name="lidar_position_x"       value="${10*cm2m}" />
+  <xacro:property name="lidar_position_z"       value="${4*cm2m}" />
   <xacro:property name="wheel_drop_offset_z"     value="${3.5*mm2m}"/>
   <xacro:property name="wheel_drop_z"            value="${wheel_height + wheel_drop_offset_z}"/>
@@ -76,5 +78,6 @@
   </xacro:caster>
   <!-- LiDAR -->
-  <xacro:lidar_sensor>
+  <xacro:lidar_sensor name="lidar" parent_link="base_link">
+    <origin xyz="${lidar_position_x} 0 ${lidar_position_z  + base_link_z_offset}" rpy="0 0 0"/>
   </xacro:lidar_sensor>
   <!-- IMU -->

File: hermes_create_description/urdf/sensors/lidar.urdf.xacro (robot description, xacro)
@@ -1,9 +1,23 @@
 <?xml version="1.0"?>
 <robot xmlns:xacro="http://www.ros.org/wiki/xacro">
-  <xacro:macro name="lidar_sensor">
-    <link name="lidar_frame">
+  <xacro:macro name="lidar_sensor" params="name parent_link *origin">
+    <xacro:property name="radius"        value="${5*cm2m}" />
+    <xacro:property name="length"        value="${4*cm2m}"/>
+    <xacro:property name="mass"          value="0.1"/>
+    <xacro:property name="min_angle"     value="-1.57"/>
+    <xacro:property name="max_angle"     value="1.57"/>
+    <xacro:property name="min_range"     value="0.1"/>
+    <xacro:property name="max_range"     value="12"/>
+    <xacro:property name="num_samples"   value="180"/>
+    <xacro:property name="update_rate"   value="10"/>
+    <joint name="${name}_joint" type="fixed">
+        <parent link="${parent_link}"/>
+        <child link="${name}_link"/>
+        <xacro:insert_block name="origin"/>
+    </joint>
+    <link name="${name}_link">
       <visual>
         <geometry>
-          <cylinder radius="0.05" length="0.04"/>
+          <cylinder radius="${radius}" length="${length}"/>
         </geometry>
         <material name="red">
@@ -13,35 +27,30 @@
       <collision>
         <geometry>
-          <cylinder radius="0.05" length="0.04"/>
+          <cylinder radius="${radius}" length="${length}"/>
         </geometry>
       </collision>
-      <xacro:inertial_cylinder mass="0.1" length="0.04" radius="0.05"/>
+      <xacro:inertial_cylinder mass="${mass}" length="${length}" radius="${radius}"/>
     </link>
-    <joint name="lidar_joint" type="fixed">
-        <parent link="base_link"/>
-        <child link="lidar_frame"/>
-        <origin xyz="0.10 0 0.108" rpy="0 0 0"/>
-    </joint>
-    <gazebo reference="lidar_frame">
+    <gazebo reference="${name}_link">
       <sensor name="laser" type="ray">
         <pose> 0 0 0 0 0 0 </pose>
         <visualize>true</visualize>
-        <update_rate>10</update_rate>
+        <update_rate>${update_rate}</update_rate>
         <ray>
           <scan>
             <horizontal>
-              <samples>360</samples>
-              <min_angle>-3.14</min_angle>
-              <max_angle>3.14</max_angle>
+              <samples>${num_samples}</samples>
+              <min_angle>${min_angle}</min_angle>
+              <max_angle>${max_angle}</max_angle>
             </horizontal>
           </scan>
           <range>
-            <min>0.1</min>
-            <max>12</max>
+            <min>${min_range}</min>
+            <max>${max_range}</max>
           </range>
         </ray>
         <plugin name="laser_controller" filename="libgazebo_ros_ray_sensor.so">
           <ros>
-            <argument>~/out:=scan</argument>
+            <remapping>~/out:=scan</remapping>
           </ros>
           <output_type>sensor_msgs/LaserScan</output_type>
