Commit message: Fixed the script issues, updated README, updated the robot package name.

File: hermes_robot_description/urdf/caster.urdf.xacro (robot description, xacro)
@@ -2,5 +2,5 @@
 <robot xmlns:xacro="http://ros.org/wiki/xacro">
 <xacro:macro name="caster" params="name parent_link *origin">
-  <xacro:include filename="$(find hermes_create_description)/urdf/common_properties.urdf.xacro"/>
+  <xacro:include filename="$(find hermes_robot_description)/urdf/common_properties.urdf.xacro"/>
   <xacro:property name="radius" value="${1*cm2m}" />
   <xacro:property name="mass"   value="0.01"/>

File: hermes_robot_description/urdf/create3.urdf.xacro (robot description, xacro)
@@ -1,15 +1,15 @@
 <?xml version="1.0" ?>
 <robot name="create3" xmlns:xacro="http://ros.org/wiki/xacro">
-  <xacro:include filename="$(find hermes_create_description)/urdf/bumper.urdf.xacro" />
-  <xacro:include filename="$(find hermes_create_description)/urdf/button.urdf.xacro" />
-  <xacro:include filename="$(find hermes_create_description)/urdf/caster.urdf.xacro" />
-  <xacro:include filename="$(find hermes_create_description)/urdf/common_properties.urdf.xacro"/>
-  <xacro:include filename="$(find hermes_create_description)/urdf/sensors/cliff_sensor.urdf.xacro"/>
-  <xacro:include filename="$(find hermes_create_description)/urdf/sensors/imu.urdf.xacro" />
-  <xacro:include filename="$(find hermes_create_description)/urdf/sensors/ir_intensity.urdf.xacro" />
-  <xacro:include filename="$(find hermes_create_description)/urdf/sensors/ir_opcode_receivers.urdf.xacro" />
-  <xacro:include filename="$(find hermes_create_description)/urdf/sensors/optical_mouse.urdf.xacro"/>
-  <xacro:include filename="$(find hermes_create_description)/urdf/sensors/lidar.urdf.xacro"/>
-  <xacro:include filename="$(find hermes_create_description)/urdf/wheel_with_wheeldrop.urdf.xacro" />
+  <xacro:include filename="$(find hermes_robot_description)/urdf/bumper.urdf.xacro" />
+  <xacro:include filename="$(find hermes_robot_description)/urdf/button.urdf.xacro" />
+  <xacro:include filename="$(find hermes_robot_description)/urdf/caster.urdf.xacro" />
+  <xacro:include filename="$(find hermes_robot_description)/urdf/common_properties.urdf.xacro"/>
+  <xacro:include filename="$(find hermes_robot_description)/urdf/sensors/cliff_sensor.urdf.xacro"/>
+  <xacro:include filename="$(find hermes_robot_description)/urdf/sensors/imu.urdf.xacro" />
+  <xacro:include filename="$(find hermes_robot_description)/urdf/sensors/ir_intensity.urdf.xacro" />
+  <xacro:include filename="$(find hermes_robot_description)/urdf/sensors/ir_opcode_receivers.urdf.xacro" />
+  <xacro:include filename="$(find hermes_robot_description)/urdf/sensors/optical_mouse.urdf.xacro"/>
+  <xacro:include filename="$(find hermes_robot_description)/urdf/sensors/lidar.urdf.xacro"/>
+  <xacro:include filename="$(find hermes_robot_description)/urdf/wheel_with_wheeldrop.urdf.xacro" />
   <!-- Mechanical properties -->
   <xacro:property name="body_z_offset"           value="${-2.5*cm2m}" />
@@ -41,5 +41,5 @@
       <origin xyz="0 0 ${body_z_offset + base_link_z_offset}" rpy="0 0 ${pi/2}"/>
       <geometry>
-        <mesh filename="file://$(find hermes_create_description)/meshes/body_visual.dae" />
+        <mesh filename="file://$(find hermes_robot_description)/meshes/body_visual.dae" />
       </geometry>
     </visual>
@@ -56,6 +56,6 @@
   <!-- Bumper -->
   <xacro:bumper
-      visual_mesh="file://$(find hermes_create_description)/meshes/bumper_visual.dae"
-      collision_mesh="file://$(find hermes_create_description)/meshes/bumper_collision.dae">
+      visual_mesh="file://$(find hermes_robot_description)/meshes/bumper_visual.dae"
+      collision_mesh="file://$(find hermes_robot_description)/meshes/bumper_collision.dae">
     <origin xyz="0 0 ${bumper_offset_z  + base_link_z_offset}"/>
     <inertial>

File: hermes_robot_description/urdf/dock/standard.urdf.xacro (robot description, xacro)
@@ -1,6 +1,6 @@
 <?xml version="1.0"?>
 <robot name="standard_dock" xmlns:xacro="http://ros.org/wiki/xacro">
-  <xacro:include filename="$(find hermes_create_description)/urdf/common_properties.urdf.xacro"/>
-  <xacro:include filename="$(find hermes_create_description)/urdf/dock/ir_emitter.urdf.xacro"/>
+  <xacro:include filename="$(find hermes_robot_description)/urdf/common_properties.urdf.xacro"/>
+  <xacro:include filename="$(find hermes_robot_description)/urdf/dock/ir_emitter.urdf.xacro"/>
   <xacro:property name="z_offset"  value="${4.6*mm2m}"/>
   <xacro:property name="link_name" value="std_dock_link"/>
@@ -9,5 +9,5 @@
       <origin xyz="0 0 ${z_offset}"/>
       <geometry>
-        <mesh filename="file://$(find hermes_create_description)/meshes/dock/visual.dae"/>
+        <mesh filename="file://$(find hermes_robot_description)/meshes/dock/visual.dae"/>
       </geometry>
     </visual>

File: hermes_robot_description/urdf/sensors/ir_intensity.urdf.xacro (robot description, xacro)
@@ -1,5 +1,5 @@
 <?xml version="1.0"?>
 <robot xmlns:xacro="http://ros.org/wiki/xacro">
-  <xacro:include filename="$(find hermes_create_description)/urdf/common_properties.urdf.xacro"/>
+  <xacro:include filename="$(find hermes_robot_description)/urdf/common_properties.urdf.xacro"/>
   <xacro:macro name="ir_intensity"
                params="name parent:=base_link

File: hermes_robot_description/urdf/wheel_drop.urdf.xacro (robot description, xacro)
@@ -2,5 +2,5 @@
 <robot xmlns:xacro="http://ros.org/wiki/xacro">
 <xacro:macro name="wheel_drop" params="name parent_link *origin" >
-  <xacro:include filename="$(find hermes_create_description)/urdf/common_properties.urdf.xacro"/>
+  <xacro:include filename="$(find hermes_robot_description)/urdf/common_properties.urdf.xacro"/>
   <xacro:property name="detection_threshold" value="${3*cm2m}"/>
   <xacro:property name="spring_stiffness_nm" value="450"/>

File: hermes_robot_description/urdf/wheel_with_wheeldrop.urdf.xacro (robot description, xacro)
@@ -2,6 +2,6 @@
 <robot xmlns:xacro="http://ros.org/wiki/xacro">
 <xacro:macro name="wheel_with_wheeldrop" params="name parent_link:=base_link *origin">
-  <xacro:include filename="$(find hermes_create_description)/urdf/wheel.urdf.xacro" />
-  <xacro:include filename="$(find hermes_create_description)/urdf/wheel_drop.urdf.xacro" />
+  <xacro:include filename="$(find hermes_robot_description)/urdf/wheel.urdf.xacro" />
+  <xacro:include filename="$(find hermes_robot_description)/urdf/wheel_drop.urdf.xacro" />
   <!-- Wheel Drop definition -->
   <xacro:wheel_drop name="${name}" parent_link="${parent_link}">
